Commit message: added the working vehicle model

File: buggy_vehicle_description/urdf/vehicle.xacro (robot description, xacro)
@@ -8,5 +8,5 @@
       <origin xyz="${vehicle_info['/**']['ros__parameters']['wheel_base']/2.0} 0 0" rpy="${pi/2.0} 0 ${pi}"/>
       <geometry>
-        <mesh filename="package://buggy_vehicle_description/mesh/buggyassembly.dae" scale="1 1 1"/>
+        <mesh filename="package://buggy_vehicle_description/mesh/buggy_8_seater_unity.stl" scale="1 1 1"/>
       </geometry>
     </visual>

Commit message: adjusted scale size

File: buggy_vehicle_description/urdf/vehicle.xacro (robot description, xacro)
@@ -8,5 +8,5 @@
       <origin xyz="${vehicle_info['/**']['ros__parameters']['wheel_base']/2.0} 0 0" rpy="${pi/2.0} 0 ${pi}"/>
       <geometry>
-        <mesh filename="package://buggy_vehicle_description/mesh/buggy_8_seater_unity.stl" scale="1 1 1"/>
+        <mesh filename="package://buggy_vehicle_description/mesh/buggy_8_seater_unity.stl" scale="0.01 0.01 0.01"/>
       </geometry>
     </visual>

Commit message: adjusted orientation

File: buggy_vehicle_description/urdf/vehicle.xacro (robot description, xacro)
@@ -6,5 +6,5 @@
   <link name="base_link">
     <visual>
-      <origin xyz="${vehicle_info['/**']['ros__parameters']['wheel_base']/2.0} 0 0" rpy="${pi/2.0} 0 ${pi}"/>
+      <origin xyz="${vehicle_info['/**']['ros__parameters']['wheel_base']/2.0} 0 0" rpy="${pi/2.0} 0 ${pi/2.0}"/>
       <geometry>
         <mesh filename="package://buggy_vehicle_description/mesh/buggy_8_seater_unity.stl" scale="0.01 0.01 0.01"/>

Commit message: Added origin fixed stl

File: buggy_vehicle_description/urdf/vehicle.xacro (robot description, xacro)
@@ -8,5 +8,5 @@
       <origin xyz="${vehicle_info['/**']['ros__parameters']['wheel_base']/2.0} 0 0" rpy="${pi/2.0} 0 ${pi/2.0}"/>
       <geometry>
-        <mesh filename="package://buggy_vehicle_description/mesh/buggy_8_seater_unity.stl" scale="0.01 0.01 0.01"/>
+        <mesh filename="package://buggy_vehicle_description/mesh/buggy_8_seater_new.stl" scale="0.01 0.01 0.01"/>
       </geometry>
     </visual>

Commit message: Added y_up stl

File: buggy_vehicle_description/urdf/vehicle.xacro (robot description, xacro)
@@ -8,5 +8,5 @@
       <origin xyz="${vehicle_info['/**']['ros__parameters']['wheel_base']/2.0} 0 0" rpy="${pi/2.0} 0 ${pi/2.0}"/>
       <geometry>
-        <mesh filename="package://buggy_vehicle_description/mesh/buggy_8_seater_new.stl" scale="0.01 0.01 0.01"/>
+        <mesh filename="package://buggy_vehicle_description/mesh/buggy_8_seater_new_yup.stl" scale="0.01 0.01 0.01"/>
       </geometry>
     </visual>
